Commit message: Minor precision fix

File: uu-robots/metralabs_ros/Models/xacro/scitos_haw_only.xacro (robot description, xacro)
@@ -3,5 +3,5 @@
 <link name="base_link"><!--Odometry origin, former called ScitosBase -->
   <visual>
-    <origin xyz="-0.075 0 0.29" rpy="0 0 0" />
+    <origin xyz="-0.075 0 ${scitos_height/2}" rpy="0 0 0" />
     <geometry>
       <cylinder radius="${scitos_width/2}" length="${scitos_height}" />
@@ -10,5 +10,5 @@
   </visual>
   <collision>
-    <origin xyz="-0.075 0 ${0.29 + 0.1/2}" rpy="0 0 0" />
+    <origin xyz="-0.075 0 ${scitos_height/2 + 0.1/2}" rpy="0 0 0" />
     <geometry>
       <cylinder radius="${scitos_width*1.2/2}" length="${scitos_height+0.1}" />

Commit message: xacro model files cleanup

File: uu-robots/metralabs_ros/Models/xacro/scitos_haw_only.xacro (robot description, xacro)
@@ -32,5 +32,5 @@
 <!-- Laserscanner, no effect beside nice to see -->
 <!--
-<link name="Laserscanner">
+<link name="laser">
   <visual>
     <origin xyz="${0.109+0.120/2} 0 ${0.326+0.120/2}"/>
@@ -41,5 +41,5 @@
   </visual>
 </link>
-<xacro:connect parent="ScitosBase" child="Laserscanner"/>
+<xacro:connect parent="scitos_base" child="laser"/>
 -->
 </robot>

File: uu-robots/metralabs_ros/Models/xacro/scitos_haw_properties.xacro (robot description, xacro)
@@ -12,6 +12,5 @@
 <xacro:property name="schunk_base_offset_rear" value="-0.252" /><!--arm mounted in rear position-->
 <!--restraint-->
-<xacro:property name="max_vel" value="0.43" /> <!--abgerundete geschwindigkeit des langsamsten gelenks-->
- <!--quark: 2.88r/s ~= 16°/s was etwa die Hälfte der mittleren Maximalgeschwindigkeit der Drehgelenke ist... halt moment, 2.88 muss Quark sein.. -->
+<xacro:property name="max_vel" value="0.43" /> <!--rounded down maximum velocity of slowest joint -->
 <!-- Materials -->
 <material name="black">

File: uu-robots/metralabs_ros/Models/xacro/scitos_haw_schunk_joints.xacro (robot description, xacro)
@@ -7,5 +7,5 @@
  <joint name="DH_1_2" type="revolute">
 	<!-- ~center of base swivel joint ID20 -->
-    <!-- the ~center means: both z of this and below added must equal 0.268 -->
+    <!-- the ~center means: both z of this and below added must equal 0.268 to match reality -->
     <origin xyz="0 0 0.120" rpy="0 0 0"/>
     <parent link="DH1"/>
@@ -110,136 +110,3 @@
  </joint>
 -->
-<!-- Backup: alle Koordinatensysteme gleich ausgerichtet:
- <joint name="DH_2_3" type="revolute">
-    <origin xyz="0 0 0.268" rpy="0 0 0"/>
-    <parent link="DH2"/>
-    <child link="DH3"/>
-    <axis xyz="0 1 0" />
-    <limit lower="-3.0543" upper="3.0543" effort="2" velocity="${max_vel}" />
- </joint>
- <joint name="DH_3_4" type="revolute">
-    <origin xyz="0 0 0.400" rpy="0 0 ${0.5*tau}"/>
-    <parent link="DH3"/>
-    <child link="DH4"/>
-    <axis xyz="0 1 0" />
-    <limit lower="-3.0543" upper="3.0543" effort="2" velocity="${max_vel}" />
- </joint>
- <joint name="DH_4_5" type="revolute">
-    <origin xyz="0 0 0.300" rpy="0 0 ${0.5*tau}"/>
-    <parent link="DH4"/>
-    <child link="DH5"/>
-    <axis xyz="0 1 0" />
-    <limit lower="-3.0543" upper="3.0543" effort="2" velocity="${max_vel}" />
- </joint>
- <joint name="DH_5_6" type="revolute">
-    <origin xyz="0 0 0.200" rpy="0 0 0"/>
-    <parent link="DH5"/>
-    <child link="DH6"/>
-    <axis xyz="0 0 1" />
-    <limit lower="-3.0543" upper="3.0543" effort="2" velocity="${max_vel}" />
- </joint>
--->
-<!--
- <joint name="Base_ConnBase" type="fixed">
-    <origin xyz="0 0 0.75" rpy="0 0 ${0.5*tau}"/>
-    <parent link="ScitosBase"/>
-    <child link="ConnBase"/>
- </joint>
- <joint name="ConnBase_J1" type="fixed">
-    <origin xyz="0 0 0.060" rpy="0 0 0"/>
-    <parent link="ConnBase"/>
-    <child link="J1"/>
- </joint>
- <joint name="J1_Conn1" type="revolute">
-    <origin xyz="0 0 0.180" rpy="${0.25*tau} 0 0"/>
-    <parent link="J1"/>
-    <child link="Conn1"/>
-    <limit lower="-3.0543" upper="3.0543" effort="2" velocity="${max_vel}" />
-    <axis xyz="0 0 1" />
- </joint>
- <joint name="Conn1_J2" type="fixed">
-    <origin xyz="0 0 0.0725" rpy="0 0 0"/>
-    <parent link="Conn1"/>
-    <child link="J2"/>
- </joint>
- <joint name="J2_Conn2" type="revolute">
-    <origin xyz="0 0 0.0725" rpy="0 0 0"/>
-    <parent link="J2"/>
-    <child link="Conn2"/>
-    <limit lower="-3.0543" upper="3.0543" effort="2" velocity="${max_vel}" />
-    <axis xyz="0 0 1" />
- </joint>
--->
-<!--
-  <joint name="Fixed_C" type="fixed">
-    <origin xyz="0 0 0.0675" rpy="0 0 0"/>
-    <parent link="PAM102"/>
-    <child link="P90_2_LowerCube"/>
- </joint>
--->
-<!--
- <joint name="Joint1" type="revolute">
-    <origin xyz="0 0.09 0" rpy="0 0 0"/>
-    <parent link="P90_2_LowerCube"/>
-    <child link="P90_2_UpperCube"/>
-    <limit lower="-2.0071" upper="2.0071" effort="2" velocity="${max_vel}" />
-    <axis xyz="0 1 0" />
- </joint>
- <joint name="Fixed_D" type="fixed">
-    <origin xyz="0 -0.00025 0.106" rpy="0 0 0"/>
-    <parent link="P90_2_UpperCube"/>
-    <child link="PAM121"/>
- </joint>
- <joint name="Fixed_E" type="fixed">
-    <origin xyz="0 -0.09025 0.016" rpy="0 0 0"/>
-    <parent link="PAM121"/>
-    <child link="P90_3_LowerCube"/>
- </joint>
- <joint name="Joint2" type="revolute">
-    <origin xyz="0 0 0.09 " rpy="0 0 0"/>
-    <parent link="P90_3_LowerCube"/>
-    <child link="P90_3_UpperCube"/>
-    <limit lower="-2.8099" upper="2.8099" effort="2" velocity="${max_vel}" />
-    <axis xyz="0 0 1" />
- </joint>
- <joint name="Fixed_F" type="fixed">
-    <origin xyz="0 0 0.0675" rpy="0 0 0"/>
-    <parent link="P90_3_UpperCube"/>
-    <child link="PAM110"/>
- </joint>
- <joint name="Fixed_G" type="fixed">
-    <origin xyz="0 0 0.0575" rpy="0 0 0"/>
-    <parent link="PAM110"/>
-    <child link="P70_1_LowerCube"/>
- </joint>
- <joint name="Joint3" type="revolute">
-    <origin xyz="0 -0.07 0 " rpy="0 0 0"/>
-    <parent link="P70_1_LowerCube"/>
-    <child link="P70_1_UpperCube"/>
-    <limit lower="-0.78539816339744828" upper="2.007" effort="2" velocity="${max_vel}" />
-    <axis xyz="0 -1 0" />
- </joint>
- <joint name="Fixed_H" type="fixed">
-    <origin xyz="0 -0.00025 0.084" rpy="0 0 0"/>
-    <parent link="P70_1_UpperCube"/>
-    <child link="PAM120"/>
- </joint>
- <joint name="Fixed_I" type="fixed">
-    <origin xyz="0 0.07025 0.014" rpy="0 0 0"/>
-    <parent link="PAM120"/>
-    <child link="P70_2_LowerCube"/>
- </joint>
- <joint name="Joint4" type="revolute">
-    <origin xyz="0  0 0.07" rpy="0 0 0"/>
-    <parent link="P70_2_LowerCube"/>
-    <child link="P70_2_UpperCube"/>
-    <limit lower="-2.8099" upper="2.8099" effort="2" velocity="${max_vel}" />
-    <axis xyz="0 0 1" />
- </joint>
- <joint name="Fixed_J" type="fixed">
-    <origin xyz="0 0 0.0525" rpy="0 0 0"/>
-    <parent link="P70_2_UpperCube"/>
-    <child link="PAM100"/>
- </joint>
--->
 </robot>

File: uu-robots/metralabs_ros/Models/xacro/scitos_haw_schunk_links.xacro (robot description, xacro)
@@ -4,13 +4,15 @@
 <xacro:macro name="DH" params="name">
 <link name="${name}">
-  <!--- -><visual>
+  <!-- - ->
+  <visual>
     <geometry>
       <cylinder radius="0.030" length="0.100"/>
     </geometry>
     <material name="black"/>
-  </visual><!- - -->
+  </visual>
+  <!- - -->
 </link>
 </xacro:macro>
-<!-- -->
+<!-- schunk PRL model joint -->
 <xacro:macro name="PRL" params="name type">
 <link name="${name}" >
@@ -28,5 +30,5 @@
 </link>
 </xacro:macro>
-<!-- orthogonal connector -->
+<!-- general connector with definable shape -->
 TODO: remove macro? or disable collision in another way
 <xacro:macro name="Connector" params="name *shape">
@@ -39,11 +41,14 @@
     <material name="black"/>
   </visual>
-<!--  <collision>
+<!--
+  <collision>
     <geometry>
       <xacro:insert_block name="shape" />
     </geometry>
-  </collision>-->
+  </collision>
+-->
 </link>
 </xacro:macro>
+<!-- long flat connector between joints -->
 <xacro:macro name="Connector_long" params="name length">
 <link name="${name}" >
