Commit message: Fixed arm length, added camera mount and kinect.

File: uu-robots/metralabs_ros/Models/scitos_haw_schunk.urdf (robot description, URDF)
Before this commit: robot scitos_haw_schunk, 15 links, 14 joints
Links:
- added link Kinect; collision box size=0.08 0.30 0.06; visual box size=0.06 0.28 0.04
- link CameraMount: geometry collision box size=0.090 0.070 0.030; visual box size=0.073 0.051 0.025
Joints:
- added joint CameraMount_Kinect: type fixed, parent CameraMount, child Kinect, origin xyz=-0.015 0 0.04 rpy=0 0 0
- joint DH_5_6: origin xyz=0.107 0 0 rpy=0 1.57079632679 0 -> xyz=0.121 0 0 rpy=0 1.57079632679 0
- joint DH_6_GR: origin xyz=0 0 0.110 rpy=0 -1.57079632679 0 -> xyz=0 0 0.130 rpy=0 -1.57079632679 0
- joint GR_Fneg: origin xyz=0 0 0 rpy=0 0 0 -> xyz=0.047 0 0 rpy=0 0 0
- joint Gripper_CameraMount: origin xyz=-0.020 -0.055 0 rpy=0 0 0 -> xyz=-0.011 -0.055 0 rpy=1.57079632679 0 0

File: uu-robots/metralabs_ros/Models/xacro/scitos_haw_schunk.xacro (robot description, xacro)
@@ -41,6 +41,7 @@
 <link name="CameraMount">
   <visual>
+    <origin xyz="-0.0085 0 -0.003210" rpy="0 0 0" />
     <geometry>
-        <box size="0.075 0.020 0.055" /><!-- Werte aufrundend vermessen -->
+        <box size="0.073 0.051 0.025" /><!-- Werte vermessen -->
     </geometry>
     <material name="black"/>
@@ -48,8 +49,22 @@
   <collision>
     <geometry>
-        <box size="0.090 0.030 0.070" />
+        <box size="0.090 0.070  0.030" />
     </geometry>
   </collision>
 </link>
-<xacro:connect_xyz parent="Gripper" child="CameraMount" xyz="-0.020 -0.055 0"/><!-- Werte grob vermessen/berechnet -->
+<xacro:connect_xyz_rpy parent="Gripper" child="CameraMount" xyz="-0.011 -0.055 0" rpy="${0.25*tau} 0 0"/><!-- Werte berechnet -->
+<link name="Kinect">
+  <visual>
+    <geometry>
+        <box size="0.06 0.28 0.04" /><!-- Werte auf cm vermessen -->
+    </geometry>
+    <material name="black"/>
+  </visual>
+  <collision>
+    <geometry>
+        <box size="0.08 0.30 0.06" />
+    </geometry>
+  </collision>
+</link>
+<xacro:connect_xyz parent="CameraMount" child="Kinect" xyz="-0.015 0 0.04"/><!-- Werte auf cm vermessen -->
 </robot>

File: uu-robots/metralabs_ros/Models/xacro/scitos_haw_schunk_joints.xacro (robot description, xacro)
@@ -40,5 +40,5 @@
  <joint name="DH_5_6" type="revolute">
 	<!-- center of hand roll joint ID24 -->
-    <origin xyz="0.107 0 0" rpy="0 ${0.25*tau} 0"/>
+    <origin xyz="0.121 0 0" rpy="0 ${0.25*tau} 0"/>
     <parent link="DH5"/>
     <child link="DH6"/>
@@ -47,5 +47,5 @@
  </joint>
  <joint name="DH_6_GR" type="fixed">
-    <origin xyz="0 0 0.110" rpy="0 ${-0.25*tau} 0"/>
+    <origin xyz="0 0 0.130" rpy="0 ${-0.25*tau} 0"/>
     <parent link="DH6"/>
     <child link="Gripper"/>
@@ -59,5 +59,5 @@
  </joint>
  <joint name="GR_Fneg" type="prismatic">
-    <origin xyz="0 0 0" rpy="0 0 0"/>
+    <origin xyz="0.047 0 0" rpy="0 0 0"/>
     <parent link="Gripper"/>
     <child link="GFneg"/>

File: uu-robots/metralabs_ros/Models/xacro/scitos_haw_schunk_links.xacro (robot description, xacro)
@@ -67,5 +67,5 @@
     <visual>
     <!--<origin xyz="${0.047+0.035} 0 ${reflect*(gripper_space+0.010)/2}"/>-->
-        <origin xyz="${0.047+0.035} 0 ${1*0.020/2}"/> <!--offsets to set fingers ontop the gripper and beside the coordinate center-->
+        <origin xyz="${0.035} 0 ${1*0.020/2}"/> <!--offsets to set fingers ontop the gripper and beside the coordinate center-->
         <geometry>
             <box size="0.070 0.030 0.020"/> <!--real finger size-->

Commit message: Entered exact joint speeds

File: uu-robots/metralabs_ros/Models/scitos_haw_schunk.urdf (robot description, URDF)
Before this commit: robot scitos_haw_schunk, 16 links, 15 joints
Joints:
- joint DH_1_2: limit lower=-3.141593 upper=3.141593 effort=2 velocity=0.43 -> lower=-3.141593 upper=3.141593 effort=2 velocity=0.437
- joint DH_2_3: limit lower=-2.024580 upper=2.024580 effort=2 velocity=0.43 -> lower=-2.024580 upper=2.024580 effort=2 velocity=0.438
- joint DH_3_4: limit lower=-2.740166 upper=2.740166 effort=2 velocity=0.43 -> lower=-2.740166 upper=2.740166 effort=2 velocity=0.436
- joint DH_4_5: limit lower=-2.373644 upper=2.286380 effort=2 velocity=0.43 -> lower=-2.373644 upper=2.286380 effort=2 velocity=0.486
- joint DH_5_6: limit lower=-3.143321 upper=3.143321 effort=2 velocity=0.43 -> lower=-3.143321 upper=3.143321 effort=2 velocity=0.872

File: uu-robots/metralabs_ros/Models/xacro/scitos_haw_schunk_joints.xacro (robot description, xacro)
@@ -12,5 +12,5 @@
     <child link="DH2"/>
     <axis xyz="0 0 -1" />
-    <limit lower="-3.141593" upper="3.141593" effort="2" velocity="${max_vel}" />
+    <limit lower="-3.141593" upper="3.141593" effort="2" velocity="0.437" />
  </joint>
  <joint name="DH_2_3" type="revolute">
@@ -20,5 +20,5 @@
     <child link="DH3"/>
     <axis xyz="0 0 -1" />
-    <limit lower="-2.024580" upper="2.024580" effort="2" velocity="${max_vel}" />
+    <limit lower="-2.024580" upper="2.024580" effort="2" velocity="0.438" />
  </joint>
  <joint name="DH_3_4" type="revolute">
@@ -28,5 +28,5 @@
     <child link="DH4"/>
     <axis xyz="0 0 -1" />
-    <limit lower="-2.740166" upper="2.740166" effort="2" velocity="${max_vel}" />
+    <limit lower="-2.740166" upper="2.740166" effort="2" velocity="0.436" />
  </joint>
  <joint name="DH_4_5" type="revolute">
@@ -36,5 +36,5 @@
     <child link="DH5"/>
     <axis xyz="0 0 -1" />
-    <limit lower="-2.373644" upper="2.286380" effort="2" velocity="${max_vel}" />
+    <limit lower="-2.373644" upper="2.286380" effort="2" velocity="0.486" />
  </joint>
  <joint name="DH_5_6" type="revolute">
@@ -44,5 +44,5 @@
     <child link="DH6"/>
     <axis xyz="0 0 -1" />
-    <limit lower="-3.143321" upper="3.143321" effort="2" velocity="${max_vel}" />
+    <limit lower="-3.143321" upper="3.143321" effort="2" velocity="0.872" />
  </joint>
  <joint name="DH_6_GR" type="fixed">
